File: Hardware/AVRinator.kicad_pcb (KiCad board)
At the start: 4 copper layers, 16.5 x 33.6 mm, 47 parts, among them J2 ICSP, J3 VCOM, J4 USB_C_Receptacle_USB2.0_16P, SW1 BOOT0, U1 STM32G431K8Ux, U2 STM32G431K8Tx, U3 AP2112K-3.3, U4 AP2112K-3.3, U5 USBLC6-2SC6, U6 TXS0108EPW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

Commit message: Add JLCJLCJLCJLC incantation
Other:
- board text added: "JLCJLCJLCJLC"
Changed lines of the file:
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@@
+		)
+	)
+	(gr_text "JLCJLCJLCJLC"
+		(at 56.0832 61.6204 90)
+		(layer "F.SilkS")
+		(effects
+			(font
+				(size 0.8 0.8)
+				(thickness 0.15)
+			)
+			(justify left bottom)
 		)
 	)

Commit message: Update pin naming
Connections:
- net /USB_SBU1 renamed /SWDIO
- net /USB_SBU2 renamed /SWCLK
- net /VCOM_CTS renamed /A
- net /VCOM_CTS_VCC renamed /A_VCC
- net /VCOM_RTS renamed /B
- net /VCOM_RTS_VCC renamed /B_VCC
