File: Hardware/AVRinator.kicad_sch (KiCad schematic)
At the start: 46 parts, among them J2 ICSP, J3 VCOM, J4 USB_C_Receptacle_USB2.0_16P, SW1 BOOT0, U1 STM32G431K8Ux, U2 STM32G431K8Tx, U3 AP2112K-3.3, U4 AP2112K-3.3, U5 USBLC6-2SC6, U6 TXS0108EPW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

Commit message: Add TXS0108EPW decoupling cap and tune skew of usb
Parts:
- added C12: 100nF, Capacitor_SMD:C_0603_1608Metric, symbol Device:C_Small
Connections:
- net GND: now also C12.2
- net T_VCC: now also C12.1
Changed lines of the file:
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@@
 	)
 	(symbol
+		(lib_id "Device:C_Small")
+		(at 167.64 26.67 0)
+		(unit 1)
+		(exclude_from_sim no)
+		(in_bom yes)
+		(on_board yes)
+		(dnp no)
+		(fields_autoplaced yes)
+		(property "Reference" "C12"
+			(at 170.18 25.4063 0)
+			(effects
+				(font
+					(size 1.27 1.27)
+				)
+				(justify left)
+			)
+		)
+		(property "Value" "100nF"
+			(at 170.18 27.9463 0)
+			(effects
+				(font
+					(size 1.27 1.27)
+				)
+				(justify left)
+			)
+		)
+		(property "Footprint" "Capacitor_SMD:C_0603_1608Metric"
+			(at 167.64 26.67 0)
+			(effects
+				(font
+					(size 1.27 1.27)
+				)
+				(hide yes)
+			)
+		)
+		(property "Datasheet" "~"
+			(at 167.64 26.67 0)
+			(effects
+				(font
+					(size 1.27 1.27)
+				)
+				(hide yes)
+			)
+		)
+		(property "Description" "Unpolarized capacitor, small symbol"
+			(at 167.64 26.67 0)
+			(effects
+				(font
+					(size 1.27 1.27)
+				)
+				(hide yes)
+			)
+		)
+		(pin "1"
+		)
+		(pin "2"
+		)
+		(instances
+			(project "AVRinator"
+				(path "/8002b462-6a40-4fb2-a1a1-f934458772f1"
+					(reference "C12")
+					(unit 1)
+				)
+			)
+		)
+	)
+	(symbol
 		(lib_id "power:GND")
 		(at 198.12 106.68 0)
@@
 	)
 	(symbol
+		(lib_id "power:VCC")
+		(at 167.64 24.13 0)
+		(unit 1)
+		(exclude_from_sim no)
+		(in_bom yes)
+		(on_board yes)
+		(dnp no)
+		(fields_autoplaced yes)
+		(property "Reference" "#PWR046"
+			(at 167.64 27.94 0)
+			(effects
+				(font
+					(size 1.27 1.27)
+				)
+				(hide yes)
+			)
+		)
+		(property "Value" "T_VCC"
+			(at 167.64 19.05 0)
+			(effects
+				(font
+					(size 1.27 1.27)
+				)
+			)
+		)
+		(property "Footprint" ""
+			(at 167.64 24.13 0)
+			(effects
+				(font
+					(size 1.27 1.27)
+				)
+				(hide yes)
+			)
+		)
+		(property "Datasheet" ""
+			(at 167.64 24.13 0)
+			(effects
+				(font
+					(size 1.27 1.27)
+				)
+				(hide yes)
+			)
+		)
+		(property "Description" "Power symbol creates a global label with name \"VCC\""
+			(at 167.64 24.13 0)
+			(effects
+				(font
+					(size 1.27 1.27)
+				)
+				(hide yes)
+			)
+		)
+		(pin "1"
+		)
+		(instances
+			(project "AVRinator"
+				(path "/8002b462-6a40-4fb2-a1a1-f934458772f1"
+					(reference "#PWR046")
+					(unit 1)
+				)
+			)
+		)
+	)
+	(symbol
 		(lib_id "power:PWR_FLAG")
 		(at 30.48 101.6 0)
@@
 					(unit 1)
 				)
+			)
+		)
+	)
+	(symbol
+		(lib_id "power:GND")
+		(at 167.64 29.21 0)
+		(unit 1)
+		(exclude_from_sim no)
+		(in_bom yes)
+		(on_board yes)
+		(dnp no)
+		(fields_autoplaced yes)
+		(property "Reference" "#PWR035"
+			(at 167.64 35.56 0)
+			(effects
+				(font
+					(size 1.27 1.27)
+				)
+				(hide yes)
+			)
+		)
+		(property "Value" "GND"
+			(at 167.64 34.29 0)
+			(effects
+				(font
+					(size 1.27 1.27)
+				)
+			)
+		)
+		(property "Footprint" ""
+			(at 167.64 29.21 0)
+			(effects
+				(font
+					(size 1.27 1.27)
+				)
+				(hide yes)
+			)
+		)
+		(property "Datasheet" ""
+			(at 167.64 29.21 0)
+			(effects
+				(font
+					(size 1.27 1.27)
+				)
+				(hide yes)
+			)
+		)
+		(property "Description" "Power symbol creates a global label with name \"GND\" , ground"
+			(at 167.64 29.21 0)
+			(effects
+				(font
+					(size 1.27 1.27)
+				)
+				(hide yes)
+			)
+		)
+		(pin "1"
+		)
+		(instances
+			(project "AVRinator"
+				(path "/8002b462-6a40-4fb2-a1a1-f934458772f1"
+					(reference "#PWR035")
+					(unit 1)
+				)

Commit message: Update pin naming
Connections:
- net USB_SBU1 renamed SWDIO
- net USB_SBU2 renamed SWCLK
- net VCOM_CTS renamed A
- net VCOM_CTS_VCC renamed A_VCC
- net VCOM_RTS renamed B
- net VCOM_RTS_VCC renamed B_VCC
Changed lines of the file:
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@@
 		)
 	)
-	(label "USB_SBU1"
+	(label "SWDIO"
 		(at 60.96 175.26 180)
 		(fields_autoplaced yes)
@@
 		)
 	)
-	(label "VCOM_CTS_VCC"
+	(label "A_VCC"
 		(at 248.92 48.26 0)
 		(fields_autoplaced yes)
@@
 		)
 	)
-	(label "VCOM_RTS_VCC"
+	(label "B_VCC"
 		(at 248.92 58.42 0)
 		(fields_autoplaced yes)
@@
 		)
 	)
-	(label "VCOM_RTS"
+	(label "B"
 		(at 76.2 35.56 180)
 		(fields_autoplaced yes)
@@
 		)
 	)
-	(label "USB_SBU1"
+	(label "SWDIO"
 		(at 76.2 66.04 180)
 		(fields_autoplaced yes)
@@
 		)
 	)
-	(label "USB_SBU2"
+	(label "SWCLK"
 		(at 76.2 68.58 180)
 		(fields_autoplaced yes)
@@
 		)
 	)
-	(label "USB_SBU2"
+	(label "SWCLK"
 		(at 60.96 177.8 180)
 		(fields_autoplaced yes)
@@
 		)
 	)
-	(label "VCOM_CTS"
+	(label "A"
 		(at 76.2 33.02 180)
 		(fields_autoplaced yes)
@@
 		)
 	)
-	(label "VCOM_CTS"
+	(label "A"
 		(at 121.92 50.8 0)
 		(fields_autoplaced yes)
@@
 		)
 	)
-	(label "VCOM_RTS_VCC"
+	(label "B_VCC"
 		(at 172.72 43.18 180)
 		(fields_autoplaced yes)
@@
 		)
 	)
-	(label "VCOM_CTS_VCC"
+	(label "A_VCC"
 		(at 172.72 50.8 180)
 		(fields_autoplaced yes)
@@
 		)
 	)
-	(label "VCOM_RTS"
+	(label "B"
 		(at 121.92 43.18 0)
 		(fields_autoplaced yes)
